Commit message: Tested floating kinect urdf in Gazebo, tuned kinect's parameters to what I've found online. Created a launch file floating_kinect.launch that will launch the floating kinect, the table and the racing wheel model with physics paused.

File: wpi_drc_sim/descriptions/floating_kinect.urdf (robot description, URDF)
Before this commit: robot sensor_head, 6 links, 5 joints
Joints:
- joint kinect_to_base: origin xyz=0.031 0.0 0.053 -> xyz=0.031 0.0 0.103

Commit message: Floating Kinect Changes

File: wpi_drc_sim/descriptions/floating_kinect.urdf (robot description, URDF)
Before this commit: robot sensor_head, 6 links, 5 joints
Links:
- removed link camera_depth_frame
- removed link camera_depth_optical_frame
- removed link camera_rgb_frame
- removed link camera_rgb_optical_frame
- removed link sensor_base_link
- added link kinect_depth_frame, mass 0.01
- added link kinect_depth_optical_frame, mass 0.001
- added link kinect_rgb_frame, mass 0.001
- added link kinect_rgb_optical_frame, mass 0.001
- added link kinect_sim_link, mass 0.1; collision box size=0.005 0.005 0.05; visual box size=0.005 0.005 0.05
Joints:
- removed joint camera_depth_joint
- removed joint camera_depth_optical_joint
- removed joint camera_rgb_joint
- removed joint camera_rgb_optical_joint
- added joint kinect_depth_joint: type fixed, parent kinect_link, child kinect_depth_frame, origin xyz=0 0.018 0 rpy=0 0 0
- added joint kinect_depth_optical_joint: type fixed, parent kinect_depth_frame, child kinect_depth_optical_frame, origin xyz=0 0 0 rpy=-1.570795 0 -1.570795
- added joint kinect_rgb_joint: type fixed, parent kinect_link, child kinect_rgb_frame, origin xyz=0 -0.005 0 rpy=0 0 0
- added joint kinect_rgb_optical_joint: type fixed, parent kinect_rgb_frame, child kinect_rgb_optical_frame, origin xyz=0 0 0 rpy=-1.570795 0 -1.570795
- joint kinect_to_base: parent sensor_base_link -> kinect_sim_link

Commit message: Working floating kinect

File: wpi_drc_sim/descriptions/floating_kinect.urdf (robot description, URDF)
Before this commit: robot sensor_head, 6 links, 5 joints
Joints:
- joint kinect_depth_optical_joint: origin xyz=0 0 0 rpy=-1.570795 0 -1.570795 -> xyz=0 0 0 rpy=-1.20919958 1.20919958 -1.20919958
- joint kinect_rgb_optical_joint: origin xyz=0 0 0 rpy=-1.570795 0 -1.570795 -> xyz=0 0 0 rpy=-1.20919958 1.20919958 -1.20919958
- joint kinect_to_base: origin xyz=0.031 0.0 0.103 -> xyz=0.031 0.0 0.103 rpy=0 0.78539816 0
